Commit message: actualizacion del ejercicio

File: src/urdf_tutorial-master/urdf/arm_3.urdf (robot description, URDF)
Before this commit: robot arm_3, 4 links, 3 joints
Links:
- removed link joint_2_link
- removed link joint_3_link
- added link eslabon2_link, mass 1; collision cylinder length=0.4 radius=0.06; visual cylinder length=0.3 radius=0.04
- added link eslabon3_link, mass 1; collision cylinder length=0.4 radius=0.06; visual cylinder length=0.3 radius=0.04
Joints:
- removed joint joint_2
- removed joint joint_3
- added joint eslabon2: type revolute, parent eslabon1_link, child eslabon2_link, origin xyz=0 0 0.3 rpy=0 0 1.5, axis 0 1 0, limit lower=-2.5 upper=2.5 effort=300 velocity=0.1
- added joint eslabon3: type prismatic, parent eslabon2_link, child eslabon3_link, origin xyz=0 0 0.2 rpy=0 0 1.5, axis 0 0 1, limit lower=-0.15 upper=0.04 effort=300 velocity=0.1

Commit message: ejercicio5 mejorado

File: src/urdf_tutorial-master/urdf/arm_3.urdf (robot description, URDF)
Before this commit: robot arm_3, 4 links, 3 joints
Links:
- link base_link: geometry collision cylinder length=0.05 radius=0.1; visual cylinder length=0.06 radius=0.1
- link eslabon1_link: geometry collision cylinder length=0.4 radius=0.06; visual cylinder length=0.3 radius=0.042
- link eslabon2_link: geometry collision cylinder length=0.3 radius=0.04; visual cylinder length=0.3 radius=0.04
- link eslabon3_link: geometry collision cylinder length=0.4 radius=0.06; visual cylinder length=0.3 radius=0.02
Joints:
- joint eslabon1: origin xyz=0 0 0.1 -> xyz=0 0 0.06
- joint eslabon2: origin xyz=0 0 0.3 rpy=0 0 1.5 -> xyz=0 0 0.25 rpy=0 0 0
- joint eslabon3: limit lower=-0.15 upper=0.04 effort=300 velocity=0.1 -> lower=0 upper=0.19 effort=300 velocity=0.1; origin xyz=0 0 0.2 rpy=0 0 1.5 -> xyz=0 0 0.05 rpy=0 0 0.05
